Commit message: completed teleop r2d2 tutorial

File: src/my_r2d2/urdf/r2d2.urdf (robot description, URDF)
Before this commit: robot macroed, 5 links, 4 joints
Links:
- added link base_footprint
Joints:
- added joint footprinttobase: type fixed, parent base_footprint, child base_link, origin xyz=0 0 ${wheeldiam+.05+leglen-0.25}
